File: EAGLE/v2_I2C_1602/UVBox-I2C.brd (EAGLE design)
At the start: 99.8 x 46 mm, 50 parts, among them IC1 7812DT, IC2 7805DT, IC3 IC-FT232R, IC4 ATMEGA328P, IC5 ULN2003AD, Q1 16M, SW1 Start, SW2 Mode, SW3 Add, SW4 Sub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

Commit message: 新增直接使用 LCD 結合母版的方式
Routing:
- net GND: vias 0 -> 7
Changed lines of the file:
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@@
 <?xml version="1.0" encoding="utf-8"?>
 <!DOCTYPE eagle SYSTEM "eagle.dtd">
-<eagle version="7.5.0">
+<eagle version="7.6.0">
 <drawing>
 <settings>
@@
 <param name="mdViaViaSameLayer" value="8mil"/>
 <param name="mnLayersViaInSmd" value="2"/>
-<param name="mdCopperDimension" value="20mil"/>
+<param name="mdCopperDimension" value="10mil"/>
 <param name="mdDrill" value="8mil"/>
 <param name="mdSmdStop" value="0mil"/>
 <param name="msWidth" value="10mil"/>
-<param name="msDrill" value="0.3mm"/>
+<param name="msDrill" value="10mil"/>
 <param name="msMicroVia" value="9.99mm"/>
 <param name="msBlindViaRatio" value="0.5"/>
@@
 <param name="mlMinStopFrame" value="4mil"/>
 <param name="mlMaxStopFrame" value="4mil"/>
-<param name="mlMinCreamFrame" value="0mil"/>
+<param name="mlMinCreamFrame" value="4mil"/>
 <param name="mlMaxCreamFrame" value="0mil"/>
 <param name="mlViaStopLimit" value="0mil"/>
@@
 <param name="srMinRoundness" value="0mil"/>
 <param name="srMaxRoundness" value="0mil"/>
-<param name="slThermalIsolate" value="16mil"/>
-<param name="slThermalsForVias" value="1"/>
+<param name="slThermalIsolate" value="10mil"/>
+<param name="slThermalsForVias" value="0"/>
 <param name="dpMaxLengthDifference" value="10mm"/>
 <param name="dpGapFactor" value="2.5"/>
@@
 </elements>
 <signals>
-<signal name="GND">
+<signal name="GND" airwireshidden="yes">
 <contactref element="C8" pad="1"/>
 <contactref element="ICSP" pad="6"/>
@@
 <wire x1="86.868" y1="33.02" x2="88.98" y2="33.02" width="0.6096" layer="16"/>
 <wire x1="88.98" y1="33.02" x2="89" y2="33.04" width="0.254" layer="16"/>
-<polygon width="0.254" layer="1" isolate="0.4064" orphans="yes">
+<polygon width="0.254" layer="1" orphans="yes">
 <vertex x="99.822" y="42.721215625"/>
 <vertex x="99.822" y="3.0585625" curve="-90"/>
@@
 <wire x1="93.472" y1="30.48" x2="90.678" y2="33.02" width="0.6096" layer="1"/>
 <wire x1="90.678" y1="33.02" x2="89.02" y2="33.02" width="0.6096" layer="1"/>
-<polygon width="0.254" layer="16" isolate="0.4064" orphans="yes">
+<polygon width="0.254" layer="16" orphans="yes">
 <vertex x="99.822" y="42.721215625"/>
 <vertex x="99.822" y="3.0585625" curve="-90"/>
@@
 <wire x1="42.17039375" y1="22.49639375" x2="42.17039375" y2="22.48539375" width="0.4064" layer="1"/>
 <wire x1="42.17039375" y1="22.48539375" x2="42.164" y2="22.479" width="0.4064" layer="1"/>
+<via x="28.956" y="20.32" extent="1-16" drill="0.381"/>
+<via x="34.036" y="12.954" extent="1-16" drill="0.381"/>
+<via x="45.974" y="22.86" extent="1-16" drill="0.381"/>
+<via x="48.26" y="16.51" extent="1-16" drill="0.381"/>
+<via x="34.798" y="35.306" extent="1-16" drill="0.381"/>
+<via x="45.72" y="35.306" extent="1-16" drill="0.381"/>
+<via x="85.09" y="7.366" extent="1-16" drill="0.381"/>
 </signal>
 <signal name="N$9">

Commit message: 細微修改
Routing:
- net GND: track 378.7 -> 11.5 mm, vias 7 -> 25
- net TX: track 30.3 -> 28.5 mm
